Commit message: Added gz hooks to g1.urdf, fixed g1 stl links and gz environment path, added hrc_msgs pkg to hold cpp custom msgs/srv definitions.

File: hrc_handler/urdf/g1.urdf (robot description, URDF)
Before this commit: robot g1, 44 links, 43 joints
Links:
- link head_link: geometry collision mesh filename=package://hrc_handler/meshes/g1/head_link.STL; visual mesh filename=package://hrc_handler/meshes/g1/head_link.STL
- link left_ankle_pitch_link: geometry collision mesh filename=package://hrc_handler/meshes/g1/left_ankle_pitch_link.STL; visual mesh filename=package://hrc_handler/meshes/g1/left_ankle_pitch_link.STL
- link left_ankle_roll_link: geometry collision mesh filename=package://hrc_handler/meshes/g1/left_ankle_roll_link.STL; visual mesh filename=package://hrc_handler/meshes/g1/left_ankle_roll_link.STL
- link left_elbow_pitch_link: geometry collision mesh filename=package://hrc_handler/meshes/g1/left_elbow_pitch_link.STL; visual mesh filename=package://hrc_handler/meshes/g1/left_elbow_pitch_link.STL
- link left_elbow_roll_link: geometry collision mesh filename=package://hrc_handler/meshes/g1/left_elbow_roll_link.STL; visual mesh filename=package://hrc_handler/meshes/g1/left_elbow_roll_link.STL
- link left_five_link: geometry collision mesh filename=package://hrc_handler/meshes/g1/left_five_link.STL; visual mesh filename=package://hrc_handler/meshes/g1/left_five_link.STL
- link left_four_link: geometry collision mesh filename=package://hrc_handler/meshes/g1/left_four_link.STL; visual mesh filename=package://hrc_handler/meshes/g1/left_four_link.STL
- link left_hip_pitch_link: geometry collision mesh filename=package://hrc_handler/meshes/g1/left_hip_pitch_link.STL; visual mesh filename=package://hrc_handler/meshes/g1/left_hip_pitch_link.STL
- link left_hip_roll_link: geometry collision mesh filename=package://hrc_handler/meshes/g1/left_hip_roll_link.STL; visual mesh filename=package://hrc_handler/meshes/g1/left_hip_roll_link.STL
- link left_hip_yaw_link: geometry collision mesh filename=package://hrc_handler/meshes/g1/left_hip_yaw_link.STL; visual mesh filename=package://hrc_handler/meshes/g1/left_hip_yaw_link.STL
- link left_knee_link: geometry collision cylinder length=0.15 radius=0.015; visual mesh filename=package://hrc_handler/meshes/g1/left_knee_link.STL
- link left_one_link: geometry collision box size=0.02 0.03 0.02; visual mesh filename=package://hrc_handler/meshes/g1/left_one_link.STL
- link left_palm_link: geometry collision mesh filename=package://hrc_handler/meshes/g1/left_palm_link.STL; visual mesh filename=package://hrc_handler/meshes/g1/left_palm_link.STL
- link left_shoulder_pitch_link: geometry collision mesh filename=package://hrc_handler/meshes/g1/left_shoulder_pitch_link.STL; visual mesh filename=package://hrc_handler/meshes/g1/left_shoulder_pitch_link.STL
- link left_shoulder_roll_link: geometry collision cylinder length=0.03 radius=0.03; visual mesh filename=package://hrc_handler/meshes/g1/left_shoulder_roll_link.STL
- link left_shoulder_yaw_link: geometry collision mesh filename=package://hrc_handler/meshes/g1/left_shoulder_yaw_link.STL; visual mesh filename=package://hrc_handler/meshes/g1/left_shoulder_yaw_link.STL
- link left_six_link: geometry collision mesh filename=package://hrc_handler/meshes/g1/left_six_link.STL; visual mesh filename=package://hrc_handler/meshes/g1/left_six_link.STL
- link left_three_link: geometry collision mesh filename=package://hrc_handler/meshes/g1/left_three_link.STL; visual mesh filename=package://hrc_handler/meshes/g1/left_three_link.STL
- link left_two_link: geometry collision mesh filename=package://hrc_handler/meshes/g1/left_two_link.STL; visual mesh filename=package://hrc_handler/meshes/g1/left_two_link.STL
- link left_zero_link: geometry visual mesh filename=package://hrc_handler/meshes/g1/left_zero_link.STL
- link logo_link: geometry collision mesh filename=package://hrc_handler/meshes/g1/logo_link.STL; visual mesh filename=package://hrc_handler/meshes/g1/logo_link.STL
- link pelvis: geometry collision mesh filename=package://hrc_handler/meshes/g1/pelvis.STL; visual mesh filename=package://hrc_handler/meshes/g1/pelvis.STL
- link pelvis_contour_link: geometry visual mesh filename=package://hrc_handler/meshes/g1/pelvis_contour_link.STL
- link right_ankle_pitch_link: geometry collision mesh filename=package://hrc_handler/meshes/g1/right_ankle_pitch_link.STL; visual mesh filename=package://hrc_handler/meshes/g1/right_ankle_pitch_link.STL
- link right_ankle_roll_link: geometry collision mesh filename=package://hrc_handler/meshes/g1/right_ankle_roll_link.STL; visual mesh filename=package://hrc_handler/meshes/g1/right_ankle_roll_link.STL
- link right_elbow_pitch_link: geometry collision mesh filename=package://hrc_handler/meshes/g1/right_elbow_pitch_link.STL; visual mesh filename=package://hrc_handler/meshes/g1/right_elbow_pitch_link.STL
- link right_elbow_roll_link: geometry collision mesh filename=package://hrc_handler/meshes/g1/right_elbow_roll_link.STL; visual mesh filename=package://hrc_handler/meshes/g1/right_elbow_roll_link.STL
- link right_five_link: geometry collision mesh filename=package://hrc_handler/meshes/g1/right_five_link.STL; visual mesh filename=package://hrc_handler/meshes/g1/right_five_link.STL
- link right_four_link: geometry collision mesh filename=package://hrc_handler/meshes/g1/right_four_link.STL; visual mesh filename=package://hrc_handler/meshes/g1/right_four_link.STL
- link right_hip_pitch_link: geometry collision mesh filename=package://hrc_handler/meshes/g1/right_hip_pitch_link.STL; visual mesh filename=package://hrc_handler/meshes/g1/right_hip_pitch_link.STL
- link right_hip_roll_link: geometry collision mesh filename=package://hrc_handler/meshes/g1/right_hip_roll_link.STL; visual mesh filename=package://hrc_handler/meshes/g1/right_hip_roll_link.STL
- link right_hip_yaw_link: geometry collision mesh filename=package://hrc_handler/meshes/g1/right_hip_yaw_link.STL; visual mesh filename=package://hrc_handler/meshes/g1/right_hip_yaw_link.STL
- link right_knee_link: geometry collision cylinder length=0.15 radius=0.015; visual mesh filename=package://hrc_handler/meshes/g1/right_knee_link.STL
- link right_one_link: geometry collision box size=0.02 0.03 0.02; visual mesh filename=package://hrc_handler/meshes/g1/right_one_link.STL
- link right_palm_link: geometry collision mesh filename=package://hrc_handler/meshes/g1/right_palm_link.STL; visual mesh filename=package://hrc_handler/meshes/g1/right_palm_link.STL
- link right_shoulder_pitch_link: geometry collision mesh filename=package://hrc_handler/meshes/g1/right_shoulder_pitch_link.S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; visual mesh filename=package://hrc_handler/meshes/g1/right_shoulder_pitch_link.S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
- link right_shoulder_roll_link: geometry collision cylinder length=0.03 radius=0.03; visual mesh filename=package://hrc_handler/meshes/g1/right_shoulder_roll_link.STL
- link right_shoulder_yaw_link: geometry collision mesh filename=package://hrc_handler/meshes/g1/right_shoulder_yaw_link.STL; visual mesh filename=package://hrc_handler/meshes/g1/right_shoulder_yaw_link.STL
- link right_six_link: geometry collision mesh filename=package://hrc_handler/meshes/g1/right_six_link.STL; visual mesh filename=package://hrc_handler/meshes/g1/right_six_link.STL
- link right_three_link: geometry collision mesh filename=package://hrc_handler/meshes/g1/right_three_link.STL; visual mesh filename=package://hrc_handler/meshes/g1/right_three_link.STL
- link right_two_link: geometry collision mesh filename=package://hrc_handler/meshes/g1/right_two_link.STL; visual mesh filename=package://hrc_handler/meshes/g1/right_two_link.STL
- link right_zero_link: geometry visual mesh filename=package://hrc_handler/meshes/g1/right_zero_link.STL
- link torso_link: geometry collision mesh filename=package://hrc_handler/meshes/g1/torso_link.STL; visual mesh filename=package://hrc_handler/meshes/g1/torso_link.STL

Commit message: com shift

File: hrc_handler/urdf/g1.urdf (robot description, URDF)
Before this commit: robot g1, 44 links, 43 joints
Links:
- link left_ankle_roll_link: geometry collision box size=0.25234 0.08704 0.05874; visual mesh filename=package://hrc_handler/meshes/g1/left_ankle_roll_link.STL
- link right_ankle_roll_link: geometry collision box size=0.25234 0.08704 0.05874; visual mesh filename=package://hrc_handler/meshes/g1/right_ankle_roll_link.STL

File: hrc_handler/urdf/g1_meshless.urdf (robot description, URDF)
Before this commit: robot g1, 44 links, 43 joints
Links:
- link left_ankle_roll_link: geometry collision box size=0.20234 0.05704 0.05874; visual sphere radius=0.01
- link right_ankle_roll_link: geometry collision box size=0.20234 0.05704 0.05874; visual sphere radius=0.01
